File: hardware/experiments/solenoid_driver/solenoid_driver.kicad_pcb (KiCad board)
At the start: 2 copper layers, 78 x 82.5 mm, 28 parts, among them Q1 IRLZ44N, Q2 IRLZ44N, Q3 IRLZ44N, Q4 IRLZ44N

Commit message: feat: in-line fuse on PCB (#7)
Parts:
- added F1: 7.5A, Fuse:Fuseholder_Blade_Mini_Keystone_3568, F.Cu at (73.0, 51.8)
- moved POWER_SUPPLY1 14.5 mm to (91.7, 52.6)
- moved D5 6.17 mm to (108.0, 49.5)
- moved R9 6.17 mm to (104.2, 58.0)
Connections:
- POWER_SUPPLY1 pad 1: +12V -> Net-(POWER_SUPPLY1-Pin_1)
Routing:
- net +12V: track 147.8 -> 183.5 mm
- net Net-(POWER_SUPPLY1-Pin_1): track 0.00 -> 13.3 mm
