File: hardware/experiments/solenoid_driver/solenoid_driver.kicad_sch (KiCad schematic)
At the start: 24 parts, among them Q1 IRLZ44N, Q2 IRLZ44N, Q3 IRLZ44N, Q4 IRLZ44N

Commit message: feat: in-line fuse on PCB (#7)
Parts:
- added F1: 7.5A, Fuse:Fuseholder_Blade_Mini_Keystone_3568, symbol Device:Fuse
Connections:
- net +12V: now also F1.1; no longer POWER_SUPPLY1.1 (Pin_1)
- new net: F1.2, POWER_SUPPLY1.1 (Pin_1)
Other:
- moved on the sheet: D5, POWER_SUPPLY1, R9
